Commit message: Added realsense to the description

File: ROS_packages/turtlebot3_mecanum_description/urdf/turtlebot3_mecanum.urdf.xacro (robot description, xacro)
@@ -55,5 +55,5 @@
         <cylinder length="0.018" radius="0.033"/>
       </geometry>
-      <material name="dark"/>
+      <material name="white"/>
     </visual>
     <collision>
@@ -84,5 +84,5 @@
         <cylinder length="0.018" radius="0.033"/>
       </geometry>
-      <material name="dark"/>
+      <material name="white"/>
     </visual>
     <collision>
@@ -113,5 +113,5 @@
         <cylinder length="0.018" radius="0.033"/>
       </geometry>
-      <material name="dark"/>
+      <material name="white"/>
     </visual>
     <collision>
@@ -142,5 +142,5 @@
         <cylinder length="0.018" radius="0.033"/>
       </geometry>
-      <material name="dark"/>
+      <material name="white"/>
     </visual>
     <collision>
@@ -194,10 +194,10 @@
   </link>
   <!-- CAMERA -->
-  <joint name="camera_joint" type="fixed">
+  <joint name="camera_rgb_joint_base" type="fixed">
     <origin xyz="0.073 -0.011 0.084" rpy="0 0 0"/>
     <parent link="base_link"/>
-    <child link="camera_link"/>
-  </joint>
-  <link name="camera_link">
+    <child link="camera_rgb_link"/>
+  </joint>
+  <link name="camera_rgb_link">
     <collision>
       <origin xyz="0.005 0.011 0.013" rpy="0 0 0"/>
@@ -209,5 +209,5 @@
   <joint name="camera_rgb_joint" type="fixed">
     <origin xyz="0.003 0.011 0.009" rpy="0 0 0"/>
-    <parent link="camera_link"/>
+    <parent link="camera_rgb_link"/>
     <child link="camera_rgb_frame"/>
   </joint>
@@ -219,3 +219,29 @@
   </joint>
   <link name="camera_rgb_optical_frame"/>
+  <!-- RGBD RealSense Camera -->
+  <joint name="realsense_base_joint" type="fixed">
+    <parent link="base_link"/>
+    <child link="base_realsense"/>
+    <origin xyz="0.039 0.0 0.093" rpy="0 0 0"/>
+  </joint>
+  <link name="base_realsense">
+    <visual name="">
+      <origin xyz="0.0 0.0 0.0215" rpy="0.0 0.0 0.0"/>
+      <geometry>
+        <cylinder radius="0.0115" length="0.043"/>
+      </geometry>
+      <material name="white"/>
+    </visual>
+    <collision>
+      <origin xyz="0.0 0.0 0.0" rpy="0.0 0.0 0.0"/>
+      <geometry>
+        <cylinder radius="0.0115" length="0.043"/>
+      </geometry>
+    </collision>
+  </link>
+  <xacro:arg name="use_nominal_extrinsics" default="true" />
+  <xacro:include filename="$(find realsense2_description)/urdf/_d435i.urdf.xacro"/>
+  <xacro:sensor_d435i parent="base_realsense" use_nominal_extrinsics="$(arg use_nominal_extrinsics)">
+    <origin xyz="0 0 0.043" rpy="0 0 0"/>
+  </xacro:sensor_d435i>
 </robot>
